File: cad/pcb/main_board/_autosave-main_board.kicad_pcb (KiCad board)
At the start: 4 copper layers, 71 parts, among them J1 USB_B_Micro, SW1 SW_DIP_x02, SW2 SW_DIP_x01, U1 STM32F401R_B-C_Tx, U2 TLV75533PDQNR

Commit message: Add Aisler files
Routing:
- added copper zone on In1.Cu, net VSS
- added copper zone on In2.Cu, net VSS
Changed lines of the file:
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@@
   (layers
     (0 "F.Cu" signal)
-    (1 "In1.Cu" power)
-    (2 "In2.Cu" power)
+    (1 "In1.Cu" power "F.VSS")
+    (2 "In2.Cu" power "B.VSS")
     (31 "B.Cu" signal)
     (32 "B.Adhes" user "B.Adhesive")
@@
   (setup
     (stackup
-      (layer "F.SilkS" (type "Top Silk Screen"))
+      (layer "F.SilkS" (type "Top Silk Screen") (color "White"))
       (layer "F.Paste" (type "Top Solder Paste"))
-      (layer "F.Mask" (type "Top Solder Mask") (thickness 0.01))
+      (layer "F.Mask" (type "Top Solder Mask") (color "Green") (thickness 0.025))
       (layer "F.Cu" (type "copper") (thickness 0.035))
-      (layer "dielectric 1" (type "prepreg") (thickness 0.1) (material "FR4") (epsilon_r 4.5) (loss_tangent 0.02))
+      (layer "dielectric 1" (type "prepreg") (color "FR4 natural") (thickness 0.14) (material "R-1551") (epsilon_r 1) (loss_tangent 0))
       (layer "In1.Cu" (type "copper") (thickness 0.035))
-      (layer "dielectric 2" (type "core") (thickness 1.24) (material "FR4") (epsilon_r 4.5) (loss_tangent 0.02))
+      (layer "dielectric 2" (type "core") (color "FR4 natural") (thickness 1.13) (material "R-1551") (epsilon_r 1) (loss_tangent 0))
       (layer "In2.Cu" (type "copper") (thickness 0.035))
-      (layer "dielectric 3" (type "prepreg") (thickness 0.1) (material "FR4") (epsilon_r 4.5) (loss_tangent 0.02))
+      (layer "dielectric 3" (type "prepreg") (color "FR4 natural") (thickness 0.14) (material "R-1551") (epsilon_r 1) (loss_tangent 0))
       (layer "B.Cu" (type "copper") (thickness 0.035))
-      (layer "B.Mask" (type "Bottom Solder Mask") (thickness 0.01))
+      (layer "B.Mask" (type "Bottom Solder Mask") (color "Green") (thickness 0.025))
       (layer "B.Paste" (type "Bottom Solder Paste"))
-      (layer "B.SilkS" (type "Bottom Silk Screen"))
+      (layer "B.SilkS" (type "Bottom Silk Screen") (color "White"))
       (copper_finish "None")
       (dielectric_constraints no)
@@
     )
   )
+  (zone (net 2) (net_name "VSS") (layer "In1.Cu") (hatch edge 0.5)
+    (connect_pads (clearance 0.5))
+    (min_thickness 0.25) (filled_areas_thickness no)
+    (fill yes (thermal_gap 0.5) (thermal_bridge_width 0.5))
+    (polygon
+      (pts
+        (xy 35 25)
+        (xy 225 25)
+        (xy 225 165)
+        (xy 35 165)
+      )
+    )
+  )
+  (zone (net 2) (net_name "VSS") (layer "In2.Cu") (hatch edge 0.5)
+    (priority 1)
+    (connect_pads (clearance 0.5))
+    (min_thickness 0.25) (filled_areas_thickness no)
+    (fill yes (thermal_gap 0.5) (thermal_bridge_width 0.5))
+    (polygon
+      (pts
+        (xy 35 25)
+        (xy 225 25)
+        (xy 225 165)
+        (xy 35 165)
+      )
+    )
+  )
