File: cad/opamp_spice/opamp_spice.kicad_sch (KiCad schematic)
At the start: 14 parts, among them U1 ${SIM.PARAMS}, U2 ${SIM.PARAMS}

Commit message: Spice simulations and switching to two TC's per module
Other:
- note added: ".op .step temp -20 80 1"
- note added: "SPICE simulation indicates: 0.471 T_{out} @ 0 mV 3.07 T_{out} @ 200mV"
- note removed: "SPICE simulation indicates: 0.471 T_{out} @ 0 mV 3.107 T_{out} @ 200mV"
Changed lines of the file:
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@@
 		)
 	)
-	(text "SPICE simulation indicates:\n0.471 T_{out} @ 0  mV\n3.107 T_{out} @ 200mV\n"
+	(text "SPICE simulation indicates:\n0.471 T_{out} @ 0  mV\n3.07  T_{out} @ 200mV\n"
 		(exclude_from_sim no)
 		(at 236.22 39.37 0)
@@
 		(effects
 			(font
+				(size 1.27 1.27)
+			)
+			(justify left top)
+		)
+	)
+	(text ".op\n.step temp -20 80 1"
+		(exclude_from_sim no)
+		(at 147.32 48.26 0)
+		(effects
+			(font
